File: Hardware/NiceDiceDIP/NiceDiceDIP.sch (KiCad schematic (older format))
At the start: 21 parts, among them J1 AVR-ISP-6, J2 Power, SW1 SW_Push_Dual, U1 ATtiny13A-PU, U2 74HC595

Commit message: В схеме DIP версии прописаны все футпринты
Parts:
- D1, D2, D3, D4, D5, D6, D7: footprint (none) -> LED_THT:LED_D5.0mm_FlatTop
- J1: footprint (none) -> Connector_PinHeader_2.54mm:PinHeader_2x03_P2.54mm_Vertical
- J2: footprint (none) -> TerminalBlock_Phoenix:TerminalBlock_Phoenix_MPT-0,5-2-2.54_1x02_P2.54mm_Horizontal
- R1, R2, R3, R4, R5, R6, R7, R8, R9: footprint (none) -> Resistor_THT:R_Axial_DIN0411_L9.9mm_D3.6mm_P5.08mm_Vertical
- SW1: footprint (none) -> Button_Switch_THT:SW_PUSH_6mm_H7.3mm
- U2: footprint (none) -> Package_DIP:DIP-16_W7.62mm
Changed lines of the file:
@@
 F 0 "D1" H 7800 1750 50  0000 C CNN
 F 1 "LED" H 7793 1686 50  0001 C CNN
-F 2 "" H 7800 1850 50  0001 C CNN
+F 2 "LED_THT:LED_D5.0mm_FlatTop" H 7800 1850 50  0001 C CNN
 F 3 "~" H 7800 1850 50  0001 C CNN
 	1    7800 1850
@@
 F 0 "D2" H 7800 2050 50  0000 C CNN
 F 1 "LED" H 7793 1986 50  0001 C CNN
-F 2 "" H 7800 2150 50  0001 C CNN
+F 2 "LED_THT:LED_D5.0mm_FlatTop" H 7800 2150 50  0001 C CNN
 F 3 "~" H 7800 2150 50  0001 C CNN
 	1    7800 2150
@@
 F 0 "D3" H 7800 2350 50  0000 C CNN
 F 1 "LED" H 7793 2286 50  0001 C CNN
-F 2 "" H 7800 2450 50  0001 C CNN
+F 2 "LED_THT:LED_D5.0mm_FlatTop" H 7800 2450 50  0001 C CNN
 F 3 "~" H 7800 2450 50  0001 C CNN
 	1    7800 2450
@@
 F 0 "D4" H 7800 2650 50  0000 C CNN
 F 1 "LED" H 7793 2586 50  0001 C CNN
-F 2 "" H 7800 2750 50  0001 C CNN
+F 2 "LED_THT:LED_D5.0mm_FlatTop" H 7800 2750 50  0001 C CNN
 F 3 "~" H 7800 2750 50  0001 C CNN
 	1    7800 2750
@@
 F 0 "D5" H 7800 2950 50  0000 C CNN
 F 1 "LED" H 7793 2886 50  0001 C CNN
-F 2 "" H 7800 3050 50  0001 C CNN
+F 2 "LED_THT:LED_D5.0mm_FlatTop" H 7800 3050 50  0001 C CNN
 F 3 "~" H 7800 3050 50  0001 C CNN
 	1    7800 3050
@@
 F 0 "D6" H 7800 3250 50  0000 C CNN
 F 1 "LED" H 7793 3186 50  0001 C CNN
-F 2 "" H 7800 3350 50  0001 C CNN
+F 2 "LED_THT:LED_D5.0mm_FlatTop" H 7800 3350 50  0001 C CNN
 F 3 "~" H 7800 3350 50  0001 C CNN
 	1    7800 3350
@@
 F 0 "D7" H 7800 3550 50  0000 C CNN
 F 1 "LED" H 7793 3486 50  0001 C CNN
-F 2 "" H 7800 3650 50  0001 C CNN
+F 2 "LED_THT:LED_D5.0mm_FlatTop" H 7800 3650 50  0001 C CNN
 F 3 "~" H 7800 3650 50  0001 C CNN
 	1    7800 3650
@@
 F 0 "R3" V 7250 1750 50  0000 C CNN
 F 1 "330" V 7250 1950 50  0000 C CNN
-F 2 "" V 7280 1850 50  0001 C CNN
+F 2 "Resistor_THT:R_Axial_DIN0411_L9.9mm_D3.6mm_P5.08mm_Vertical" V 7280 1850 50  0001 C CNN
 F 3 "~" H 7350 1850 50  0001 C CNN
 	1    7350 1850
@@
 F 0 "R4" V 7250 2050 50  0000 C CNN
 F 1 "330" V 7250 2250 50  0000 C CNN
-F 2 "" V 7280 2150 50  0001 C CNN
+F 2 "Resistor_THT:R_Axial_DIN0411_L9.9mm_D3.6mm_P5.08mm_Vertical" V 7280 2150 50  0001 C CNN
 F 3 "~" H 7350 2150 50  0001 C CNN
 	1    7350 2150
@@
 F 0 "R5" V 7250 2350 50  0000 C CNN
 F 1 "330" V 7250 2550 50  0000 C CNN
-F 2 "" V 7280 2450 50  0001 C CNN
+F 2 "Resistor_THT:R_Axial_DIN0411_L9.9mm_D3.6mm_P5.08mm_Vertical" V 7280 2450 50  0001 C CNN
 F 3 "~" H 7350 2450 50  0001 C CNN
 	1    7350 2450
@@
 F 0 "R6" V 7250 2650 50  0000 C CNN
 F 1 "330" V 7250 2850 50  0000 C CNN
-F 2 "" V 7280 2750 50  0001 C CNN
+F 2 "Resistor_THT:R_Axial_DIN0411_L9.9mm_D3.6mm_P5.08mm_Vertical" V 7280 2750 50  0001 C CNN
 F 3 "~" H 7350 2750 50  0001 C CNN
 	1    7350 2750
@@
 F 0 "R7" V 7250 2950 50  0000 C CNN
 F 1 "330" V 7250 3150 50  0000 C CNN
-F 2 "" V 7280 3050 50  0001 C CNN
+F 2 "Resistor_THT:R_Axial_DIN0411_L9.9mm_D3.6mm_P5.08mm_Vertical" V 7280 3050 50  0001 C CNN
 F 3 "~" H 7350 3050 50  0001 C CNN
 	1    7350 3050
@@
 F 0 "R8" V 7250 3250 50  0000 C CNN
 F 1 "330" V 7250 3450 50  0000 C CNN
-F 2 "" V 7280 3350 50  0001 C CNN
+F 2 "Resistor_THT:R_Axial_DIN0411_L9.9mm_D3.6mm_P5.08mm_Vertical" V 7280 3350 50  0001 C CNN
 F 3 "~" H 7350 3350 50  0001 C CNN
 	1    7350 3350
@@
 F 0 "R9" V 7250 3550 50  0000 C CNN
 F 1 "330" V 7250 3750 50  0000 C CNN
-F 2 "" V 7280 3650 50  0001 C CNN
+F 2 "Resistor_THT:R_Axial_DIN0411_L9.9mm_D3.6mm_P5.08mm_Vertical" V 7280 3650 50  0001 C CNN
 F 3 "~" H 7350 3650 50  0001 C CNN
 	1    7350 3650
@@
 F 0 "U2" H 6200 3350 50  0000 C CNN
 F 1 "74HC595" H 6550 3350 50  0000 C CNN
-F 2 "" H 6350 2750 50  0001 C CNN
+F 2 "Package_DIP:DIP-16_W7.62mm" H 6350 2750 50  0001 C CNN
 F 3 "http://www.ti.com/lit/ds/symlink/sn74hc595.pdf" H 6350 2750 50  0001 C CNN
 	1    6350 2750
@@
 F 0 "J1" H 3471 5046 50  0000 R CNN
 F 1 "AVR-ISP-6" H 3471 4955 50  0000 R CNN
-F 2 "" V 3550 5000 50  0001 C CNN
+F 2 "Connector_PinHeader_2.54mm:PinHeader_2x03_P2.54mm_Vertical" V 3550 5000 50  0001 C CNN
 F 3 " ~" H 2525 4400 50  0001 C CNN
 	1    3800 4950
@@
 F 0 "R2" H 6170 4696 50  0000 L CNN
 F 1 "10K" H 6170 4605 50  0000 L CNN
-F 2 "" V 6030 4650 50  0001 C CNN
+F 2 "Resistor_THT:R_Axial_DIN0411_L9.9mm_D3.6mm_P5.08mm_Vertical" V 6030 4650 50  0001 C CNN
 F 3 "~" H 6100 4650 50  0001 C CNN
 	1    6100 4650
@@
 F 0 "R1" H 4420 3996 50  0000 L CNN
 F 1 "10K" H 4420 3905 50  0000 L CNN
-F 2 "" V 4280 3950 50  0001 C CNN
+F 2 "Resistor_THT:R_Axial_DIN0411_L9.9mm_D3.6mm_P5.08mm_Vertical" V 4280 3950 50  0001 C CNN
 F 3 "~" H 4350 3950 50  0001 C CNN
 	1    4350 3950
@@
 F 0 "SW1" H 6700 5093 50  0000 C CNN
 F 1 "SW_Push_Dual" H 6700 5094 50  0001 C CNN
-F 2 "" H 6700 5100 50  0001 C CNN
+F 2 "Button_Switch_THT:SW_PUSH_6mm_H7.3mm" H 6700 5100 50  0001 C CNN
 F 3 "~" H 6700 5100 50  0001 C CNN
 	1    6700 4900
@@
 F 0 "J2" H 8130 4742 50  0000 L CNN
 F 1 "Power" H 8130 4651 50  0000 L CNN
-F 2 "" H 8050 4750 50  0001 C CNN
+F 2 "TerminalBlock_Phoenix:TerminalBlock_Phoenix_MPT-0,5-2-2.54_1x02_P2.54mm_Horizontal" H 8050 4750 50  0001 C CNN
 F 3 "~" H 8050 4750 50  0001 C CNN
 	1    8050 4750

Commit message: Исправлена кнопка
Parts:
- removed SW1: SW_Push_Dual, Button_Switch_THT:SW_PUSH_6mm_H7.3mm, symbol Switch:SW_Push_Dual
- added SW1: SW_Push, Button_Switch_THT:SW_PUSH_6mm_H7.3mm, symbol Switch:SW_Push
Connections:
- net Button: now also SW1.1
- net GND: now also SW1.2
Changed lines of the file:
@@
-$EndComp
-$Comp
-L Switch:SW_Push_Dual SW1
-U 1 1 61417395
-P 6700 4900
-F 0 "SW1" H 6700 5093 50  0000 C CNN
-F 1 "SW_Push_Dual" H 6700 5094 50  0001 C CNN
-F 2 "Button_Switch_THT:SW_PUSH_6mm_H7.3mm" H 6700 5100 50  0001 C CNN
-F 3 "~" H 6700 5100 50  0001 C CNN
-	1    6700 4900
-	1    0    0    -1
 $EndComp
 $Comp
 L power:GND #PWR010
 U 1 1 614182B6
-P 7000 5250
-F 0 "#PWR010" H 7000 5000 50  0001 C CNN
-F 1 "GND" H 7005 5077 50  0000 C CNN
-F 2 "" H 7000 5250 50  0001 C CNN
-F 3 "" H 7000 5250 50  0001 C CNN
-	1    7000 5250
+P 6900 5100
+F 0 "#PWR010" H 6900 4850 50  0001 C CNN
+F 1 "GND" H 6905 4927 50  0000 C CNN
+F 2 "" H 6900 5100 50  0001 C CNN
+F 3 "" H 6900 5100 50  0001 C CNN
+	1    6900 5100
 	1    0    0    -1
 $EndComp
@@
 Connection ~ 6100 4900
 Wire Wire Line
-	6100 4900 6400 4900
-Wire Wire Line
-	6500 5100 6400 5100
-Wire Wire Line
-	6400 5100 6400 4900
-Connection ~ 6400 4900
-Wire Wire Line
-	6400 4900 6500 4900
-Wire Wire Line
-	6900 4900 7000 4900
-Wire Wire Line
-	7000 4900 7000 5100
-Wire Wire Line
-	6900 5100 7000 5100
-Connection ~ 7000 5100
-Wire Wire Line
-	7000 5100 7000 5250
+	6800 4900 6900 4900
 $Comp
 L Connector:Screw_Terminal_01x02 J2
@@
 Wire Wire Line
 	1250 7300 1250 7150
+$Comp
+L Switch:SW_Push SW1
+U 1 1 614C3AF0
+P 6600 4900
+F 0 "SW1" H 6600 5093 50  0000 C CNN
+F 1 "SW_Push" H 6600 5094 50  0001 C CNN
+F 2 "Button_Switch_THT:SW_PUSH_6mm_H7.3mm" H 6600 5100 50  0001 C CNN
+F 3 "~" H 6600 5100 50  0001 C CNN
+	1    6600 4900
+	1    0    0    -1
+$EndComp
+Wire Wire Line
+	6100 4900 6400 4900
+Wire Wire Line
+	6900 4900 6900 5100
 $EndSCHEMATC
