File: Hardware/NiceDiceDIP/NiceDiceDIP.kicad_pcb (KiCad board)
At the start: 2 copper layers, 45.7 x 62.2 mm, 21 parts, among them J1 AVR-ISP-6, J2 Power, SW1 SW_Push, U1 ATtiny13A-PU, U2 74HC595

Commit message: Закончена разводка платы
Parts:
- moved SW1 8.52 mm to (152.4, 119.4), turned to 0 degrees
- moved J1 5.68 mm to (149.9, 110.5), turned to 180 degrees
Routing:
- net GND: track 0.00 -> 277.5 mm, vias 0 -> 4
- net Net-(J1-Pad3): track 0.00 -> 61.1 mm
- net Net-(J1-Pad1): track 5.08 -> 30.3 mm, vias 0 -> 2
- net VDD: track 66.4 -> 43.6 mm, vias 0 -> 2
- net Net-(J1-Pad4): track 8.67 -> 24.4 mm
- net Net-(J1-Pad5): track 75.0 -> 82.6 mm
- net Net-(U1-Pad2): track 29.4 -> 31.7 mm
- removed copper zone on B.Cu, net GND
